File: pico_peltier.kicad_pcb (KiCad board)
At the start: 4 copper layers, 56 x 88 mm, 97 parts, among them J1 USB_C_Receptacle_USB2.0_14P, J2 Conn_02x07_Odd_Even, J3 ZJY130-2864KSWLG22, J4 Screw_Terminal_01x02, SW1 SW_Push, SW2 SW_Push, SW3 RotaryEncoder_Switch, U1 W25Q128JVS, U2 RP2350_60QFN, U3 WE-TVS-82400102, U4 LT8722AV-PBF, U5 TPSM863253RDXR, Y1 ABM8-272-T3

Commit message: finalising
Parts:
- removed REF**: KiCad-Logo_5mm_SilkScreen, Symbol:KiCad-Logo_5mm_SilkScreen
- removed REF**: OSHW-Logo_5.7x6mm_SilkScreen, Symbol:OSHW-Logo_5.7x6mm_SilkScreen
- removed REF**: Symbol_HighVoltage_Triangle_6x6mm_silkscreen, high_volt:Symbol_HighVoltage_Triangle_6x6mm_silkscreen
- removed REF**: ESD-Logo_6.6x6mm_SilkScreen, Symbol:ESD-Logo_6.6x6mm_SilkScreen
- added G***: LOGO, logo:logo_syauqi, F.Cu at (103.4, 95.3)
- J1: footprint Connector_USB:USB_C_Receptacle_GCT_USB4105-xx-A_16P_TopMnt_Horizontal -> Connector_USB:USB_C_Receptacle_JAE_DX07S016JA1R1500
- moved J1 0.50 mm to (110.5, 112.9)
Connections:
- J1 pad : (no net) -> GND
- J3 pad SH1: GND -> (no net)
- J3 pad SH2: GND -> (no net)
- SW3 pad SH: GND -> (no net)
Routing:
- net GND: track 86.0 -> 83.4 mm, vias 250 -> 264
- net /mcu_rp2354a/GPIO27_ADC1: track 37.2 -> 39.4 mm
- net /mcu_rp2354a/USB_D-: track 4.71 -> 6.25 mm
- net /mcu_rp2354a/USB_D+: track 4.72 -> 3.72 mm
- net VBUS: track 30.6 -> 31.4 mm
- net /mcu_rp2354a/USB1_D+: track 6.17 -> 6.91 mm
- net /mcu_rp2354a/USB1_D-: track 6.12 -> 6.81 mm
- net /display/OLED_SDO: track 44.0 -> 44.7 mm
- net Net-(J1-CC2): track 2.41 -> 3.04 mm
- net Net-(J1-CC1): track 2.57 -> 3.20 mm
- net /peltier_cont/SFB: track 10.6 -> 11.2 mm, vias 2 -> 62
- net /peltier_cont/SW: vias 2 -> 15
- net /peltier_cont/LDR: vias 0 -> 74
Other:
- board text added: "Design for MFL by Syauqi ALias"

Commit message: update all
Parts:
- added D4: 5.1 Vz, Diode_SMD:D_SOD-123, F.Cu at (76.2, 125.5)
- R11: value 86.6k -> 14.7k
Connections:
- J1 pad : GND -> (no net)
Routing:
- net Net-(D4-K): track 5.99 -> 8.36 mm
- net GND: track 83.4 -> 84.3 mm

Commit message: final update before fab
Parts:
- added REF**: Symbol_HighVoltage_Triangle_6x6mm_silkscreen, high_volt:Symbol_HighVoltage_Triangle_6x6mm_silkscreen, F.Cu at (91.5, 143.5)
- added REF**: ESD-Logo_6.6x6mm_SilkScreen, Symbol:ESD-Logo_6.6x6mm_SilkScreen, F.Cu at (100.9, 123.7)
- added REF**: KiCad-Logo2_6mm_SilkScreen, Symbol:KiCad-Logo2_6mm_SilkScreen, F.Cu at (92.5, 91.3)
- added REF**: OSHW-Logo_7.5x8mm_SilkScreen, Symbol:OSHW-Logo_7.5x8mm_SilkScreen, F.Cu at (103.0, 87.3)
- H1, H2, H3, H4: footprint MountingHole:MountingHole_2.7mm_M2.5 -> MountingHole:MountingHole_2.7mm_M2.5_DIN965_Pad_TopBottom
