File: 3v3_psu.kicad_sch (KiCad schematic)
At the start: 10 parts, among them J4 Screw_Terminal_01x02, U5 TPSM863253RDXR

Commit message: update all
Parts:
- added D4: 5.1 Vz, Diode_SMD:D_SOD-123, symbol Device:D_Zener
- R11: value 86.6k -> 14.7k; mouser 667-ERJ-3EKF8662V -> 603-RC0603FR-1014K7L
Connections:
- net GND: now also D4.2 (A)
- net at C35.1, R11.2, R12.1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: now also D4.1 (K)

Commit message: All
Other:
- company: (none) -> Otai Labs
- title: (none) -> 3.3V Power Supply
Changed lines of the file:
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@@
 	(generator_version "9.0")
 	(paper "A4")
+	(title_block
+		(title "3.3V Power Supply")
+		(date "2025-12-11")
+		(rev "1a")
+		(company "Otai Labs")
+		(comment 1 "Design by Syauqi Alias")
+	)
 	(text "15V input to 3.3V 3A output"
 		(exclude_from_sim no)
