File: display.kicad_sch (KiCad schematic)
At the start: 16 parts, among them J3 ZJY130-2864KSWLG22, SW3 RotaryEncoder_Switch

Commit message: finalising
Parts:
- D2: mouser (none) -> 474-COM-24837
Changed lines of the file:
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@@
+			)
+		)
+		(property "mouser" "474-COM-24837 "
+			(at 233.68 90.17 0)
+			(effects
+				(font
+					(size 1.27 1.27)
+				)
+				(hide yes)
 			)
 		)

Commit message: All
Other:
- company: (none) -> Otai Labs
- title: (none) -> Display and Encoder
Changed lines of the file:
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@@
 	(generator_version "9.0")
 	(paper "A4")
+	(title_block
+		(title "Display and Encoder")
+		(date "2025-12-11")
+		(rev "1a")
+		(company "Otai Labs")
+		(comment 1 "Design by Syauqi Alias")
+	)
 	(text "Monochrome Display 1.3\" 128x64\nSH1106G"
 		(exclude_from_sim no)
