File: mcu_rp2354a.kicad_sch (KiCad schematic)
At the start: 39 parts, among them J1 USB_C_Receptacle_USB2.0_14P, SW1 SW_Push, SW2 SW_Push, U1 W25Q128JVS, U2 RP2350_60QFN, U3 WE-TVS-82400102, Y1 ABM8-272-T3

Commit message: finalising
Parts:
- J1: footprint Connector_USB:USB_C_Receptacle_GCT_USB4105-xx-A_16P_TopMnt_Horizontal -> Connector_USB:USB_C_Receptacle_JAE_DX07S016JA1R1500; mouser (none) -> 640-USB4105-GF-A
- Y1: mouser (none) -> 815-ABM8-272-T3
Changed lines of the file:
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@@
 			)
 		)
-		(property "Footprint" "Connector_USB:USB_C_Receptacle_GCT_USB4105-xx-A_16P_TopMnt_Horizontal"
+		(property "Footprint" "Connector_USB:USB_C_Receptacle_JAE_DX07S016JA1R1500"
 			(at 59.69 58.42 0)
 			(effects
@@
 		)
 		(property "farnell" "3588205"
+			(at 55.88 58.42 0)
+			(effects
+				(font
+					(size 1.27 1.27)
+				)
+				(hide yes)
+			)
+		)
+		(property "mouser" "640-USB4105-GF-A "
 			(at 55.88 58.42 0)
 			(effects
@@
 			(at 181.61 44.45 90)
 			(effects
+				(font
+					(size 1.27 1.27)
+				)
+				(hide yes)
+			)
+		)
+		(property "mouser" "815-ABM8-272-T3 "
+			(at 181.61 44.45 90)
+			(effects

Commit message: finalising again
Parts:
- J1: mouser 640-USB4105-GF-A -> 656-DX07S016JA3R1500
Changed lines of the file:
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@@
 			)
 		)
-		(property "mouser" "640-USB4105-GF-A "
+		(property "mouser" "656-DX07S016JA3R1500 "
 			(at 55.88 58.42 0)
 			(effects

Commit message: final update before fab
Parts:
- H1, H2, H3, H4: footprint MountingHole:MountingHole_2.7mm_M2.5 -> MountingHole:MountingHole_2.7mm_M2.5_DIN965_Pad_TopBottom
Changed lines of the file:
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@@
 			)
 		)
-		(property "Footprint" "MountingHole:MountingHole_2.7mm_M2.5"
+		(property "Footprint" "MountingHole:MountingHole_2.7mm_M2.5_DIN965_Pad_TopBottom"
 			(at 285.75 52.07 0)
 			(effects
@@
 			)
 		)
-		(property "Footprint" "MountingHole:MountingHole_2.7mm_M2.5"
+		(property "Footprint" "MountingHole:MountingHole_2.7mm_M2.5_DIN965_Pad_TopBottom"
 			(at 285.75 57.15 0)
 			(effects
@@
 			)
 		)
-		(property "Footprint" "MountingHole:MountingHole_2.7mm_M2.5"
+		(property "Footprint" "MountingHole:MountingHole_2.7mm_M2.5_DIN965_Pad_TopBottom"
 			(at 285.75 62.23 0)
 			(effects
@@
 			)
 		)
-		(property "Footprint" "MountingHole:MountingHole_2.7mm_M2.5"
+		(property "Footprint" "MountingHole:MountingHole_2.7mm_M2.5_DIN965_Pad_TopBottom"
 			(at 285.75 67.31 0)
 			(effects

Commit message: All
Other:
- company: (none) -> Otai Labs
- title: (none) -> RP2350 MCU
Changed lines of the file:
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@@
 	(generator_version "9.0")
 	(paper "A3")
+	(title_block
+		(title "RP2350 MCU")
+		(date "2025-12-11")
+		(rev "1a")
+		(company "Otai Labs")
+		(comment 1 "Design by Syauqi Alias")
+	)
 	(circle
 		(center 137.16 131.445)
