File: peltier_cont.kicad_sch (KiCad schematic)
At the start: 20 parts, among them U4 LT8722AV-PBF

Commit message: All
Other:
- company: (none) -> Otai Labs
- title: (none) -> LT8722 Half Bridge Driver
Changed lines of the file:
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@@
 	(generator_version "9.0")
 	(paper "A4")
+	(title_block
+		(title "LT8722 Half Bridge Driver")
+		(date "2025-12-11")
+		(rev "1a")
+		(company "Otai Labs")
+		(comment 1 "Design by Syauqi Alias")
+	)
 	(junction
 		(at 176.53 96.52)
