File: pico_peltier.kicad_sch (KiCad schematic)
At the start: 0 parts

Commit message: All
Other:
- company: (none) -> Otai Labs
- title: (none) -> Pico Peltier TEC Overall
Changed lines of the file:
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@@
 	(generator_version "9.0")
 	(paper "A4")
+	(title_block
+		(title "Pico Peltier TEC Overall")
+		(date "2025-12-11")
+		(rev "1a")
+		(company "Otai Labs")
+		(comment 1 "Design by Syauqi Alias")
+	)
 	(wire
 		(pts
