File: pinout.kicad_sch (KiCad schematic)
At the start: 1 part, among them J2 Conn_02x07_Odd_Even

Commit message: finalising
Parts:
- J2: mouser (none) -> 571-5-534236-7
Changed lines of the file:
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@@
+			)
+		)
+		(property "mouser" "571-5-534236-7 "
+			(at 146.05 95.25 0)
+			(effects
+				(font
+					(size 1.27 1.27)
+				)
+				(hide yes)
 			)
 		)

Commit message: All
Other:
- company: (none) -> Otai Labs
- title: (none) -> Extension Port
Changed lines of the file:
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@@
 	(generator_version "9.0")
 	(paper "A4")
+	(title_block
+		(title "Extension Port")
+		(date "2025-12-11")
+		(rev "1a")
+		(company "Otai Labs")
+		(comment 1 "Design by Syauqi Alias")
+	)
 	(wire
 		(pts
