File: temp_probe.kicad_sch (KiCad schematic)
At the start: 9 parts

Commit message: All
Other:
- company: (none) -> Otai Labs
- title: (none) -> NTC 10K Probe
Changed lines of the file:
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@@
 	(generator_version "9.0")
 	(paper "A4")
+	(title_block
+		(title "NTC 10K Probe")
+		(date "2025-12-11")
+		(rev "1a")
+		(company "Otai Labs")
+		(comment 1 "Design by Syauqi Alias")
+	)
 	(text "Temp probe: cold, hot and room\n\n"
 		(exclude_from_sim no)
